File: Hardware/ESP8266BlinkerXiaoAI.kicad_pcb (KiCad board)
At the start: 2 copper layers, 24.9 x 14.6 mm, 8 parts, among them J1 Conn_02x04_Top_Bottom, M1 Motor_Servo, P1 USB_C_Plug_USB2.0, SW1 SW_Push, U1 AMS1117

Commit message: V1.2
Parts:
- moved REF** 0.05 mm to (137.9, 91.9)
