File: Hardware/ESP8266BlinkerXiaoAI.kicad_sch (KiCad schematic)
At the start: 7 parts, among them J1 Conn_02x04_Top_Bottom, M1 Motor_Servo, P1 USB_C_Plug_USB2.0, SW1 SW_Push, U1 AMS1117

Commit message: V1.2
Other:
- note added: "Open-source hardware"
- note removed: "Open Hardware"
- title: ESP8266 Blinker Lamp -> ESP826 Blinker XiaoAI
Changed lines of the file:
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@@
   (paper "A4")
   (title_block
-    (title "ESP8266 Blinker Lamp")
+    (title "ESP826 Blinker XiaoAI")
     (date "2022-03-07")
     (rev "1.0")
@@
     (stroke (width 0) (type default) (color 0 0 0 0))
   )
-  (text "Open Hardware" (at 140.97 67.31 0)
+  (text "Open-source hardware" (at 132.08 68.58 0)
     (effects (font (size 3 3) (thickness 1) bold) (justify left bottom))
   )
